File: hardware/Phantom_Daughterboard_PCB/Phantom_Daughterboard_PCB.kicad_sch (KiCad schematic)
At the start: 0 parts

Commit message: Added some subsystems
Other:
- added sheet Battery Management (bms.kicad_sch)
- added sheet ESP-32 (esp32.kicad_sch)
- added sheet Power Distribution (power_distribution.kicad_sch)
Changed lines of the file:
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@@
 	(generator_version "10.0")
 	(paper "A4")
+	(sheet
+		(at 44.45 73.66)
+		(size 33.02 11.43)
+		(exclude_from_sim no)
+		(in_bom yes)
+		(on_board yes)
+		(dnp no)
+		(fields_autoplaced yes)
+		(stroke
+			(width 0.1524)
+			(type solid)
+		)
+		(fill
+			(color 0 0 0 0)
+		)
+		(property "Sheetname" "Power Distribution"
+			(at 44.45 72.9484 0)
+			(show_name no)
+			(do_not_autoplace no)
+			(effects
+				(font
+					(size 1.27 1.27)
+				)
+				(justify left bottom)
+			)
+		)
+		(property "Sheetfile" "power_distribution.kicad_sch"
+			(at 44.45 85.6746 0)
+			(show_name no)
+			(do_not_autoplace no)
+			(effects
+				(font
+					(size 1.27 1.27)
+				)
+				(justify left top)
+			)
+		)
+		(instances
+			(project "Phantom_Daughterboard_PCB"
+				(path "/6417737e-4970-46ce-94b0-3c6d1bf91825"
+					(page "2")
+				)
+			)
+		)
+	)
+	(sheet
+		(at 86.36 73.66)
+		(size 31.75 11.43)
+		(exclude_from_sim no)
+		(in_bom yes)
+		(on_board yes)
+		(dnp no)
+		(fields_autoplaced yes)
+		(stroke
+			(width 0.1524)
+			(type solid)
+		)
+		(fill
+			(color 0 0 0 0)
+		)
+		(property "Sheetname" "Battery Management"
+			(at 86.36 72.9484 0)
+			(show_name no)
+			(do_not_autoplace no)
+			(effects
+				(font
+					(size 1.27 1.27)
+				)
+				(justify left bottom)
+			)
+		)
+		(property "Sheetfile" "bms.kicad_sch"
+			(at 86.36 85.6746 0)
+			(show_name no)
+			(do_not_autoplace no)
+			(effects
+				(font
+					(size 1.27 1.27)
+				)
+				(justify left top)
+			)
+		)
+		(instances
+			(project "Phantom_Daughterboard_PCB"
+				(path "/6417737e-4970-46ce-94b0-3c6d1bf91825"
+					(page "4")
+				)
+			)
+		)
+	)
+	(sheet
+		(at 45.72 92.71)
+		(size 30.48 10.16)
+		(exclude_from_sim no)
+		(in_bom yes)
+		(on_board yes)
+		(dnp no)
+		(fields_autoplaced yes)
+		(stroke
+			(width 0.1524)
+			(type solid)
+		)
+		(fill
+			(color 0 0 0 0)
+		)
+		(property "Sheetname" "ESP-32"
+			(at 45.72 91.9984 0)
+			(show_name no)
+			(do_not_autoplace no)
+			(effects
+				(font
+					(size 1.27 1.27)
+				)
+				(justify left bottom)
+			)
+		)
+		(property "Sheetfile" "esp32.kicad_sch"
+			(at 45.72 103.4546 0)
+			(show_name no)
+			(do_not_autoplace no)
+			(effects
+				(font
+					(size 1.27 1.27)
+				)
+				(justify left top)
+			)
+		)
+		(instances
+			(project "Phantom_Daughterboard_PCB"
+				(path "/6417737e-4970-46ce-94b0-3c6d1bf91825"
+					(page "3")
+				)
+			)
+		)
+	)
 	(sheet_instances
 		(path "/"
