File: hardware/Phantom_Daughterboard_PCB/power_distribution.kicad_sch (KiCad schematic)
At the start: 0 parts

Commit message: Added buck regulator LM5164
Parts:
- added U1: LM5164DDA, Package_SO:HSOP-8-1EP_3.9x4.9mm_P1.27mm_EP2.41x3.1mm_ThermalVias, symbol Regulator_Switching:LM5164DDA
Changed lines of the file:
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@@
 	(generator_version "10.0")
 	(paper "A3")
+	(symbol
+		(lib_id "Regulator_Switching:LM5164DDA")
+		(at 138.43 137.16 0)
+		(unit 1)
+		(body_style 1)
+		(exclude_from_sim no)
+		(in_bom yes)
+		(on_board yes)
+		(in_pos_files yes)
+		(dnp no)
+		(fields_autoplaced yes)
+		(property "Reference" "U1"
+			(at 138.43 121.92 0)
+			(show_name no)
+			(do_not_autoplace no)
+			(effects
+				(font
+					(size 1.27 1.27)
+				)
+			)
+		)
+		(property "Value" "LM5164DDA"
+			(at 138.43 124.46 0)
+			(show_name no)
+			(do_not_autoplace no)
+			(effects
+				(font
+					(size 1.27 1.27)
+				)
+			)
+		)
+		(property "Footprint" "Package_SO:HSOP-8-1EP_3.9x4.9mm_P1.27mm_EP2.41x3.1mm_ThermalVias"
+			(at 139.7 148.59 0)
+			(hide yes)
+			(show_name no)
+			(do_not_autoplace no)
+			(effects
+				(font
+					(size 1.27 1.27)
+				)
+			)
+		)
+		(property "Datasheet" "https://www.ti.com/lit/ds/symlink/lm5164.pdf?ts=1598311864250&ref_url=https%253A%252F%252Fwww.ti.com%252Fproduct%252FLM5164%253FHQS%253DTI-null-null-octopart-df-pf-null-wwe"
+			(at 130.81 128.27 0)
+			(hide yes)
+			(show_name no)
+			(do_not_autoplace no)
+			(effects
+				(font
+					(size 1.27 1.27)
+				)
+			)
+		)
+		(property "Description" "1A synchronous buck converter with ultra-low IQ, 6V - 100V input, adjustable output voltage, HSOP-8"
+			(at 138.43 137.16 0)
+			(hide yes)
+			(show_name no)
+			(do_not_autoplace no)
+			(effects
+				(font
+					(size 1.27 1.27)
+				)
+			)
+		)
+		(pin "9"
+		)
+		(pin "5"
+		)
+		(pin "2"
+		)
+		(pin "8"
+		)
+		(pin "1"
+		)
+		(pin "4"
+		)
+		(pin "7"
+		)
+		(pin "6"
+		)
+		(pin "3"
+		)
+		(instances
+			(project "Phantom_Daughterboard_PCB"
+				(path "/6417737e-4970-46ce-94b0-3c6d1bf91825/2779b52f-80ed-4f2f-8f05-b118f3c9718e"
+					(reference "U1")
+					(unit 1)
+				)
+			)
+		)
+	)
 )
